File: UnoTest/UnoTest.kicad_sch (KiCad schematic)
At the start: 19 parts, among them P1 Power, P2 Analog, P3 Digital, P4 Digital, P5 CONN_01X01, P6 CONN_01X01, P7 CONN_01X01, P8 CONN_01X01

Commit message: test added
Parts:
- added Test: Screw_Terminal_01x02, symbol Connector:Screw_Terminal_01x02
- Mz1, PushButton: value (none) -> Screw_Terminal_01x02
- UV_Sensor_1: value (none) -> Screw_Terminal_01x05
Changed lines of the file:
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@@
     (in_bom yes) (on_board yes) (fields_autoplaced)
     (property "Reference" "UV_Sensor_1" (id 0) (at 38.1 16.51 0))
-    (property "Value" "" (id 1) (at 38.1 19.05 0))
+    (property "Value" "Screw_Terminal_01x05" (id 1) (at 38.1 19.05 0))
     (property "Footprint" "" (id 2) (at 38.1 27.94 0)
       (effects (font (size 1.27 1.27)) hide)
@@
     (in_bom yes) (on_board yes) (fields_autoplaced)
     (property "Reference" "Mz1" (id 0) (at 38.1 72.39 0))
-    (property "Value" "" (id 1) (at 38.1 74.93 0))
+    (property "Value" "Screw_Terminal_01x02" (id 1) (at 38.1 74.93 0))
     (property "Footprint" "" (id 2) (at 38.1 78.74 0)
       (effects (font (size 1.27 1.27)) hide)
@@
     (in_bom yes) (on_board yes) (fields_autoplaced)
     (property "Reference" "PushButton" (id 0) (at 163.83 20.32 0))
-    (property "Value" "" (id 1) (at 163.83 22.86 0))
+    (property "Value" "Screw_Terminal_01x02" (id 1) (at 163.83 22.86 0))
     (property "Footprint" "" (id 2) (at 163.83 26.67 0)
       (effects (font (size 1.27 1.27)) hide)
@@
     (in_bom yes) (on_board yes) (fields_autoplaced)
     (property "Reference" "UV_Sensor_1" (id 0) (at 60.96 16.51 0))
-    (property "Value" "" (id 1) (at 60.96 19.05 0))
+    (property "Value" "Screw_Terminal_01x05" (id 1) (at 60.96 19.05 0))
     (property "Footprint" "" (id 2) (at 60.96 27.94 0)
       (effects (font (size 1.27 1.27)) hide)
@@
     (in_bom yes) (on_board yes) (fields_autoplaced)
     (property "Reference" "UV_Sensor_1" (id 0) (at 83.82 16.51 0))
-    (property "Value" "" (id 1) (at 83.82 19.05 0))
+    (property "Value" "Screw_Terminal_01x05" (id 1) (at 83.82 19.05 0))
     (property "Footprint" "" (id 2) (at 83.82 27.94 0)
       (effects (font (size 1.27 1.27)) hide)
@@
     (pin "4")
     (pin "5")
+  )
+  (symbol (lib_id "Connector:Screw_Terminal_01x02") (at 129.54 96.52 0) (unit 1)
+    (in_bom yes) (on_board yes) (fields_autoplaced)
+    (property "Reference" "Test" (id 0) (at 132.08 96.5199 0)
+      (effects (font (size 1.27 1.27)) (justify left))
+    )
+    (property "Value" "Screw_Terminal_01x02" (id 1) (at 132.08 99.0599 0)
+      (effects (font (size 1.27 1.27)) (justify left))
+    )
+    (property "Footprint" "" (id 2) (at 129.54 96.52 0)
+      (effects (font (size 1.27 1.27)) hide)
+    )
+    (property "Datasheet" "~" (id 3) (at 129.54 96.52 0)
+      (effects (font (size 1.27 1.27)) hide)
+    )
+    (pin "1")
+    (pin "2")
   )
   (symbol (lib_id "Connector:Screw_Terminal_01x05") (at 129.54 27.94 0) (mirror y) (unit 1)
@@
       (reference "PushButton") (unit 1) (value "Screw_Terminal_01x02") (footprint "")
     )
+    (path "/dfdaa22a-0489-48da-8a56-737e4c4366e1"
+      (reference "Test") (unit 1) (value "Screw_Terminal_01x02") (footprint "")
+    )
     (path "/26770edf-0451-46f1-9399-7bcd5300fe62"
